File: KiCad/Sodium.kicad_pcb (KiCad board)
At the start: 2 copper layers, 2 parts, among them J8 0.96

Commit message: Update KiCad files
Parts:
- removed C17: 0.1u, Capacitor_SMD:C_0603_1608Metric
- added D2: GS1010FL, Diode_SMD:D_SOD-123F, F.Cu at (151.7, 72.5)
- added M1: mark, myFoot:my_TestPoint_1mm, F.Cu at (117.3, 61.7)
- added M2: mark, myFoot:my_TestPoint_1mm, F.Cu at (130.1, 137.9)
- added M3: mark, myFoot:my_TestPoint_1mm, F.Cu at (174.5, 137.9)
- added SW1: SW1, myFoot:my_SW_PUSH_12mm, B.Cu at (169.0, 107.0)
