File: KiCad/Sodium.sch (KiCad schematic (older format))
At the start: 76 parts, among them J1 INPUT, J10 SW4_GND, J2 OUTPUT, J3 DEBUG_SWD, J7 DC_Jack, J8 0.96\"_OLED_Display_Module, J9 SW4, SW0 SW0, SW1 SW1, SW2 SW2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

Commit message: Update KiCad files
Parts:
- C1, C11, C14: footprint Capacitor_SMD:C_1206_3216Metric -> Capacitor_SMD:C_0805_2012Metric
- C12, C20: value 220u -> 100u
- D2: value MBR130LSFT1G -> GS1010FL; symbol Device:D_Schottky_Small -> Device:D_Small
- J3: value DEBUG_SWD -> DEBUG
- R13, R14: value (4.7k) -> 4.7k
- TP8: value +8.7V -> +8.2V
- U2: value PCM3060PWR -> PCM3060PW
- U3: value STM32F722RCT6 -> STM32F722RET6
- U4: value LF33CDT-TR -> NJM2391DL1-33
Connections:
- net LED_RED: now also U3.23 (PA7)
- no-connect marks 35 -> 34
Other:
- note added: "0.17W"
- note added: "0.2W"
- note added: "1W"
- note added: "MAX 200mA"
- note added: "MLAE002 Sodium Rev.E\nMar. 2021\ndrugscore.blog.fc2.com"
- note removed: "0.16W"
- note removed: "0.19W"
- note removed: "1.1W"
- note removed: "MAX 250mA"
- note removed: "MLAE002 Sodium Rev.D\nDec. 2020\ndrugscore.blog.fc2.com"
